File: Shady.kicad_sch (KiCad schematic)
At the start: 69 parts, among them J1 JACK_2P, J10 Conn_01x10_Female, J11 Conn_02x05_Odd_Even, J2 JACK_2P, J3 JACK_2P, J4 JACK_2P, J5 JACK_2P, J6 JACK_2P, J7 Conn_01x10_Male, J8 Conn_01x10_Male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

Commit message: updates for rev101
Parts:
- R26, R27, R28: value 33K -> 1K
Other:
- note added: "LED resistors R26,27,28 can be 1K to 10K depending on how bright you like them"
Changed lines of the file:
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@@
     (stroke (width 0) (type default) (color 0 0 0 0))
+  )
+  (text "LED resistors R26,27,28 can be 1K to 10K\ndepending on how bright you like them"
+    (at 338.455 182.88 0)
+    (effects (font (size 1.27 1.27)) (justify left bottom))
   )
   (text "Face / Rear" (at 37.465 43.18 0)
@@
     (in_bom yes) (on_board yes)
     (property "Reference" "R28" (id 0) (at 338.455 197.3072 90))
-    (property "Value" "33K" (id 1) (at 338.455 199.6186 90))
+    (property "Value" "1K" (id 1) (at 338.455 199.6186 90))
     (property "Footprint" "Resistor_THT:R_Axial_DIN0207_L6.3mm_D2.5mm_P2.54mm_Vertical" (id 2) (at 338.455 200.787 90)
       (effects (font (size 1.27 1.27)) hide)
@@
     (in_bom yes) (on_board yes)
     (property "Reference" "R27" (id 0) (at 336.55 19.5072 90))
-    (property "Value" "33K" (id 1) (at 336.55 21.8186 90))
+    (property "Value" "1K" (id 1) (at 336.55 21.8186 90))
     (property "Footprint" "Resistor_THT:R_Axial_DIN0207_L6.3mm_D2.5mm_P2.54mm_Vertical" (id 2) (at 336.55 22.987 90)
       (effects (font (size 1.27 1.27)) hide)
@@
     (in_bom yes) (on_board yes)
     (property "Reference" "R26" (id 0) (at 344.805 109.0422 90))
-    (property "Value" "33K" (id 1) (at 344.805 111.3536 90))
+    (property "Value" "1K" (id 1) (at 344.805 111.3536 90))
     (property "Footprint" "Resistor_THT:R_Axial_DIN0207_L6.3mm_D2.5mm_P2.54mm_Vertical" (id 2) (at 344.805 112.522 90)
       (effects (font (size 1.27 1.27)) hide)
@@
     )
     (path "/c84eaf9d-5abe-4349-8093-0970633b0a50"
-      (reference "R26") (unit 1) (value "33K") (footprint "Resistor_THT:R_Axial_DIN0207_L6.3mm_D2.5mm_P2.54mm_Vertical")
+      (reference "R26") (unit 1) (value "1K") (footprint "Resistor_THT:R_Axial_DIN0207_L6.3mm_D2.5mm_P2.54mm_Vertical")
     )
     (path "/62f8f19c-ac9d-486e-be49-d1823ecfae61"
-      (reference "R27") (unit 1) (value "33K") (footprint "Resistor_THT:R_Axial_DIN0207_L6.3mm_D2.5mm_P2.54mm_Vertical")
+      (reference "R27") (unit 1) (value "1K") (footprint "Resistor_THT:R_Axial_DIN0207_L6.3mm_D2.5mm_P2.54mm_Vertical")
     )
     (path "/2e1d3295-411c-4b57-8b8a-6e6b61e2957a"
-      (reference "R28") (unit 1) (value "33K") (footprint "Resistor_THT:R_Axial_DIN0207_L6.3mm_D2.5mm_P2.54mm_Vertical")
+      (reference "R28") (unit 1) (value "1K") (footprint "Resistor_THT:R_Axial_DIN0207_L6.3mm_D2.5mm_P2.54mm_Vertical")
     )
     (path "/00000000-0000-0000-0000-00005fb6ae8f"
