File: Shady.kicad_pcb (KiCad board)
At the start: 2 copper layers, 112.4 x 128.5 mm, 89 parts, among them J1 JACK_2P, J10 Conn_01x10_Female, J11 Conn_02x05_Odd_Even, J2 JACK_2P, J3 JACK_2P, J4 JACK_2P, J5 JACK_2P, J6 JACK_2P, J7 Conn_01x10_Male, J8 Conn_01x10_Male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

Commit message: updates for rev101
Changed lines of the file:
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@@
       (drillshape 0)
       (scaleselection 1)
-      (outputdirectory "gbr")
+      (outputdirectory "gbr2")
     )
   )
@@
   (gr_line (start 63.55 39.25) (end 35.55 39.25) (layer "B.SilkS") (width 0.12))
   (gr_line (start 35.55 143.75) (end 63.55 143.75) (layer "B.SilkS") (width 0.12))
-  (gr_arc (start 47.514076 51.978811) (mid 54.94 39.35) (end 62.254076 52.048811) (layer "F.SilkS") (width 0.66))
+  (gr_arc (start 47.514076 51.978811) (mid 54.944217 39.350019) (end 62.254076 52.048811) (layer "F.SilkS") (width 0.66))
   (gr_line (start 54.95 47.85) (end 47.45 40.35) (layer "F.SilkS") (width 0.66))
   (gr_line (start 54.95 87.25) (end 62.45 79.75) (layer "F.SilkS") (width 0.66))

Commit message: v111
v111 has some triangles on the faceplate
Other:
- board text added: "Shady v1.1.1 karltron.com Derived from Mutable Instruments' Shades KDS2022-04-25"
- board text removed: "Shady v1.0.1 karltron.com Derived from Mutable Instruments' Shades KDS2022-04-25"
- board text removed: "UNTESTED"
Changed lines of the file:
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@@
   (title_block
     (title "Shady")
-    (date "2022-04-22")
-    (rev "v1.0.1")
+    (date "2022-06-02")
+    (rev "v1.1.1")
     (company "karltron.com")
     (comment 1 "based on Mutable Shades v4")
@@
       (drillshape 0)
       (scaleselection 1)
-      (outputdirectory "gbr2")
+      (outputdirectory "gbr0")
     )
   )
@@
   (gr_arc (start 47.514076 51.978811) (mid 54.944217 39.350019) (end 62.254076 52.048811) (layer "F.SilkS") (width 0.66))
   (gr_line (start 54.95 47.85) (end 47.45 40.35) (layer "F.SilkS") (width 0.66))
+  (gr_poly
+    (pts
+      (xy 37.55 75.541584)
+      (xy 37.55 74.191584)
+      (xy 39.2 74.191584)
+    ) (layer "F.SilkS") (width 0.1) (fill solid))
+  (gr_poly
+    (pts
+      (xy 37.55 95)
+      (xy 37.55 93.65)
+      (xy 39.2 93.65)
+    ) (layer "F.SilkS") (width 0.1) (fill solid))
   (gr_line (start 54.95 87.25) (end 62.45 79.75) (layer "F.SilkS") (width 0.66))
   (gr_line (start 54.95 67.55) (end 47.45 60.05) (layer "F.SilkS") (width 0.66))
   (gr_line (start 54.95 67.55) (end 62.45 60.05) (layer "F.SilkS") (width 0.66))
+  (gr_poly
+    (pts
+      (xy 40.85 82)
+      (xy 37.55 82)
+      (xy 40.85 79.85)
+    ) (layer "F.SilkS") (width 0.12) (fill solid))
+  (gr_poly
+    (pts
+      (xy 37.55 55.7)
+      (xy 37.55 54.35)
+      (xy 39.2 54.35)
+    ) (layer "F.SilkS") (width 0.1) (fill solid))
+  (gr_poly
+    (pts
+      (xy 40.85 74.191584)
+      (xy 39.2 74.191584)
+      (xy 40.85 72.841584)
+    ) (layer "F.SilkS") (width 0.1) (fill solid))
   (gr_line (start 54.95 87.25) (end 47.45 79.75) (layer "F.SilkS") (width 0.66))
   (gr_line (start 54.95 47.85) (end 62.45 40.35) (layer "F.SilkS") (width 0.66))
+  (gr_poly
+    (pts
+      (xy 40.85 54.35)
+      (xy 39.2 54.35)
+      (xy 40.85 53)
+    ) (layer "F.SilkS") (width 0.1) (fill solid))
+  (gr_poly
+    (pts
+      (xy 40.85 93.65)
+      (xy 39.2 93.65)
+      (xy 40.85 92.3)
+    ) (layer "F.SilkS") (width 0.1) (fill solid))
   (gr_arc (start 47.54 91.42) (mid 54.992658 78.737802) (end 62.29 91.51) (layer "F.SilkS") (width 0.66))
+  (gr_poly
+    (pts
+      (xy 40.85 42.7)
+      (xy 37.55 42.7)
+      (xy 40.85 40.55)
+    ) (layer "F.SilkS") (width 0.12) (fill solid))
+  (gr_poly
+    (pts
+      (xy 40.85 62.55)
+      (xy 37.55 62.55)
+      (xy 40.85 60.4)
+    ) (layer "F.SilkS") (width 0.12) (fill solid))
   (gr_arc (start 47.57 71.76) (mid 54.969584 59.044247) (end 62.3 71.8) (layer "F.SilkS") (width 0.66))
   (gr_line (start 35.55 162.75) (end 35.55 25.05) (layer "Dwgs.User") (width 0.15))
   (gr_line (start 33.35 39.25) (end 220.85 39.25) (layer "Dwgs.User") (width 0.15))
   (gr_line (start 104.55 25) (end 104.55 158.75) (layer "Dwgs.User") (width 0.15))
+  (gr_line (start 40.85 39.65) (end 40.85 97.6) (layer "Dwgs.User") (width 0.1))
   (gr_line (start 16.6 155.75) (end 225.8 155.75) (layer "Dwgs.User") (width 0.15))
   (gr_line (start 103.55 158.8) (end 103.55 25.4) (layer "Dwgs.User") (width 0.15))
@@
     (effects (font (size 1 1) (thickness 0.15)) (justify mirror))
   )
-  (gr_text "Shady v1.0.1 karltron.com\nDerived from \nMutable Instruments' Shades\nKDS2022-04-25" (at 49.45 98.6) (layer "B.SilkS")
+  (gr_text "Shady v1.1.1 karltron.com\nDerived from \nMutable Instruments' Shades\nKDS2022-04-25" (at 49.45 98.6) (layer "B.SilkS")
     (effects (font (size 1.25 1.25) (thickness 0.25)) (justify mirror))
   )
@@
     (effects (font (size 3 2.5) (thickness 0.6)))
   )
-  (gr_text "UNTESTED" (at 100.75 25.45) (layer "Cmts.User")
-    (effects (font (size 5 5) (thickness 1)))
-  )
   (dimension (type aligned) (layer "Dwgs.User")

Commit message: update to v121
switched the switches around so it matches original better
adjusted logos on front panel
Parts:
- moved G1 88.1 mm to (86.9, 42.6), turned to 180 degrees
- moved G3 0.19 mm to (78.7, 130.1)
- moved JP3 0.18 mm to (86.8, 84.7)
- moved Q1 0.11 mm to (88.0, 100.8)
- moved R3 0.05 mm to (84.8, 75.8)
- turned SW1 to -90 degrees
- turned SW2 to -90 degrees
- turned SW3 to -90 degrees
Connections:
- RV1 pad : (no net) -> GND
- RV2 pad : (no net) -> GND
- RV3 pad : (no net) -> GND
Routing:
- net GND: track 168.3 -> 161.2 mm, vias 55 -> 59
- net SS1t: track 13.0 -> 20.1 mm
- net SS2t: track 17.9 -> 11.8 mm
- net SS3t: track 35.8 -> 31.3 mm
Other:
- board text added: "Shady v1.2.1 PCB1"
- board text added: "V101 back panel compat w/ v121 front panels"
- board text added: "check position of jumper pins"
- board text added: "karltron.com Shady v1.2.1 Derived from Mutable Instruments' Shades"
- board text added: "v101 KDS2022-04-25 v121 KDS2022-10-04"
- board text removed: "Shady v1.0.1 PCB1"
- board text removed: "Shady v1.1.1 karltron.com Derived from Mutable Instruments' Shades KDS2022-04-25"
